File: Schematics/Pico_Sensor_Array/Pico_Sensor_Array.kicad_sch (KiCad schematic)
At the start: 6 parts, among them P1 Pico W

Commit message: Updated README and Demo video, added schematic
Parts:
- D1: value DHT11 -> DHT22
- RTC1: value DS1307+ -> DS1307
Changed lines of the file:
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@@
     (in_bom yes) (on_board yes)
     (property "Reference" "RTC1" (id 0) (at 106.68 103.6193 0))
-    (property "Value" "DS1307+" (id 1) (at 106.68 101.6 0))
+    (property "Value" "DS1307" (id 1) (at 106.68 101.6 0))
     (property "Footprint" "Package_DIP:DIP-8_W7.62mm" (id 2) (at 99.06 100.33 0)
       (effects (font (size 1.27 1.27)) hide)
@@
       (effects (font (size 1.27 1.27)) (justify right))
     )
-    (property "Value" "DHT11" (id 1) (at 87.63 87.6299 0)
+    (property "Value" "DHT22" (id 1) (at 87.63 87.6299 0)
       (effects (font (size 1.27 1.27)) (justify right))
     )
@@
     )
     (path "/fb1dad8f-8fc5-4d24-9f54-cdbdc7f495ca"
-      (reference "D1") (unit 1) (value "DHT11") (footprint "Sensor:Aosong_DHT11_5.5x12.0_P2.54mm")
+      (reference "D1") (unit 1) (value "DHT22") (footprint "Sensor:Aosong_DHT11_5.5x12.0_P2.54mm")
     )
     (path "/c61d9cfd-3c6c-4cef-b391-3c91f4c112fa"
@@
     )
     (path "/c0ff83d0-1efb-414c-9a85-df15e9264609"
-      (reference "RTC1") (unit 1) (value "DS1307+") (footprint "Package_DIP:DIP-8_W7.62mm")
+      (reference "RTC1") (unit 1) (value "DS1307") (footprint "Package_DIP:DIP-8_W7.62mm")
     )
     (path "/24fe6738-bcab-4c17-a742-3dfbdd5dd12c"
